File: corne-chocolate/pcb/corne-chocolate.kicad_pcb (KiCad board)
At the start: 2 copper layers, 133.8 x 91.4 mm, 98 parts, among them J3 LED, P1 i2c-pin, P2 i2c-pin, SW1 SW_PUSH, SW10 SW_PUSH, SW11 SW_PUSH, SW12 SW_PUSH, SW13 SW_PUSH, SW14 SW_PUSH, SW15 SW_PUSH, SW16 SW_PUSH, SW17 SW_PUSH, SW18 SW_PUSH, SW19 SW_PUSH, SW2 SW_PUSH, SW20 SW_PUSH, SW21 SW_PUSH, SW3 SW_PUSH, SW4 SW_PUSH, SW5 SW_PUSH, SW6 SW_PUSH, SW7 SW_PUSH, SW8 SW_PUSH, SW9 SW_PUSH, U1 ProMicro

Commit message: chocolate ready to go with extra connectors for travelling
Parts:
- removed the ? at (79.5, 105.5)
- removed the ? at (79.5, 86.8)
- removed L1, L10, L11, L12, L13, L14, L15, L16, L17, L18, L19, L2, L20, L21, L3, L4, L5, L6, L7, L8, L9: SK6812MINI, kbd:SK6812MINI_rev
- added J4: Conn_01x02, Connector_AMASS:AMASS_XT60-F_1x02_P7.20mm_Vertical, F.Cu at (189.1, 62.8)
- added J5: Conn_01x02, Connector_AMASS:AMASS_XT60-F_1x02_P7.20mm_Vertical, F.Cu at (54.5, 111.8)
- JP1: renamed from data; footprint kbd:JPC2 -> kbd:Jumper
- RSW1: value Reset -> SW_PUSH
- turned JP1 to 180 degrees
- turned JP2 to 90 degrees
- turned JP3 to 90 degrees
- turned JP4 to 90 degrees
- turned JP5 to 90 degrees
- turned JP6 to 90 degrees
- turned JP7 to 90 degrees
- turned JP8 to 90 degrees
- turned JP9 to 90 degrees
- renumbered TRRS to J1, OLED to J2
Connections:
- JP1 pad 1: data -> Net-(J1-PadB)
- JP1 pad 2: Net-(J1-PadB) -> data
- JP2 pad 1: GND -> Net-(J2-Pad4)
- JP2 pad 2: Net-(J2-Pad4) -> GND
- JP3 pad 1: VCC -> Net-(J2-Pad3)
- JP3 pad 2: Net-(J2-Pad3) -> VCC
- JP4 pad 1: SCL -> Net-(J2-Pad2)
- JP4 pad 2: Net-(J2-Pad2) -> SCL
- JP5 pad 1: SDA -> Net-(J2-Pad1)
- JP5 pad 2: Net-(J2-Pad1) -> SDA
- JP6 pad 1: SDA -> Net-(J2-Pad4)
- JP6 pad 2: Net-(J2-Pad4) -> SDA
- JP7 pad 1: SCL -> Net-(J2-Pad3)
- JP7 pad 2: Net-(J2-Pad3) -> SCL
- JP8 pad 1: VCC -> Net-(J2-Pad2)
- JP8 pad 2: Net-(J2-Pad2) -> VCC
- JP9 pad 1: GND -> Net-(J2-Pad1)
- JP9 pad 2: Net-(J2-Pad1) -> GND
- L27 pad 1: Net-(L21-Pad3) -> unconnected-(L27-Pad1)
- U1 pad 11: Net-(U1-Pad11) -> unconnected-(U1-Pad11)
- U1 pad 12: Net-(U1-Pad12) -> unconnected-(U1-Pad12)
- U1 pad 13: Net-(U1-Pad13) -> unconnected-(U1-Pad13)
- U1 pad 14: Net-(U1-Pad14) -> unconnected-(U1-Pad14)
- U1 pad 24: Net-(U1-Pad24) -> unconnected-(U1-Pad24)
Routing:
- net GND: track 816.7 -> 412.9 mm, vias 59 -> 13
- net VCC: track 786.4 -> 389.0 mm, vias 30 -> 12
- net Net-(L17-Pad1): track 48.0 -> 0.00 mm, vias 4 -> 0
- net Net-(L2-Pad3): track 46.2 -> 0.00 mm, vias 6 -> 0
- net Net-(L14-Pad1): track 45.6 -> 0.00 mm, vias 4 -> 0
- net Net-(L10-Pad1): track 42.9 -> 0.00 mm, vias 4 -> 0
- net Net-(L15-Pad3): track 41.9 -> 0.00 mm, vias 4 -> 0
- net Net-(L3-Pad1): track 40.9 -> 0.00 mm, vias 4 -> 0
- net Net-(L11-Pad3): track 40.6 -> 0.00 mm, vias 4 -> 0
- net Net-(L11-Pad1): track 40.4 -> 0.00 mm, vias 4 -> 0
- net Net-(L10-Pad3): track 39.7 -> 0.00 mm, vias 4 -> 0
- net Net-(L16-Pad3): track 39.3 -> 0.00 mm, vias 4 -> 0
- net Net-(L18-Pad3): track 39.1 -> 0.00 mm, vias 6 -> 0
- net Net-(L1-Pad1): track 38.5 -> 0.00 mm, vias 4 -> 0
- net Net-(L12-Pad1): track 37.0 -> 0.00 mm, vias 6 -> 0
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- removed copper zone on B.Cu, net GND
- removed copper zone on F.Cu, net GND
Other:
- board size 133.8 x 91.4 mm -> 145.7 x 94.9 mm
- net class Default removed
